File: gpsdo/gpsdo.kicad_pcb (KiCad board)
At the start: 2 copper layers, 100 x 100 mm, 54 parts, among them J1 Conn_02x05_Odd_Even, J2 Barrel_Jack_Switch, J3 Conn_01x04_Male, J4 USB_B_Micro, J5 Conn_01x02_Male, J6 Conn_01x06_Male, SW1 pushbutton_switch, SW2 SW_SPDT, U1 STM32F407VETx, U2 ATGM336H-5N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

Commit message: layout
Parts:
- removed J3: Conn_01x04_Male, Connector_PinHeader_2.54mm:PinHeader_1x04_P2.54mm_Vertical
- removed J6: Conn_01x06_Male, Connector_PinHeader_2.54mm:PinHeader_1x06_P2.54mm_Vertical
- added AE2: Antenna_Shield, pace:sma, F.Cu at (2.10, 50.0)
- added AE3: Antenna_Shield, pace:sma, F.Cu at (2.10, 61.9)
- added AE4: Antenna_Shield, pace:sma, F.Cu at (97.8, 73.9)
- added AE5: Antenna_Shield, pace:sma, F.Cu at (2.10, 85.8)
- added AE6: Antenna_Shield, pace:sma, F.Cu at (97.8, 50.0)
- added AE7: Antenna_Shield, pace:sma, F.Cu at (97.8, 61.9)
- added AE8: Antenna_Shield, pace:sma, F.Cu at (2.10, 73.9)
- added AE9: Antenna_Shield, pace:sma, F.Cu at (97.8, 85.8)
- added C18: 12pf, Capacitor_SMD:C_0402_1005Metric, F.Cu at (47.8, 37.0)
- added C19: 12pf, Capacitor_SMD:C_0402_1005Metric, F.Cu at (53.3, 37.0)
- added R9: 220, Resistor_SMD:R_0402_1005Metric, F.Cu at (51.0, 33.5)
- added Y1: 16mhz, Crystal:Crystal_SMD_3225-4Pin_3.2x2.5mm, F.Cu at (50.6, 36.6)
- D1: value ledgreen -> ledgreen_0805; footprint LED_SMD:LED_0603_1608Metric -> LED_SMD:LED_0805_2012Metric
- U4: value 74AHC1G04 -> 74AHC1G04-newfp; footprint Package_TO_SOT_SMD:SOT-353_SC-70-5 -> pace:SOT-70-dck
- U5: value SRV05-4 -> SRV05-4-newfp; footprint Package_TO_SOT_SMD:SOT-23-6 -> pace:srv05-4
- moved SW1 34.8 mm to (41.1, 39.9), turned to 180 degrees
- moved H4 34.1 mm to (96.6, 96.5)
- moved H3 31.1 mm to (3.40, 96.1)
- moved R2 29.6 mm to (37.8, 25.4)
- moved C1 29.6 mm to (40.7, 32.9)
- moved J1 29.1 mm to (39.0, 10.1), turned to 180 degrees
- moved R3 29.0 mm to (37.8, 23.2)
- moved R4 16.9 mm to (31.7, 32.9), turned to 0 degrees
- moved TH1 12.3 mm to (31.6, 31.3), turned to 180 degrees
- moved C12 8.28 mm to (17.0, 4.00), turned to 0 degrees
- moved TP1 7.18 mm to (37.2, 30.1)
- moved R6 6.76 mm to (36.9, 27.9)
- moved C11 5.66 mm to (77.0, 33.6), turned to 270 degrees
- moved TP2 4.75 mm to (14.3, 9.74)
- moved R5 4.65 mm to (61.9, 32.8)
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Connections:
- U1 pad 12: /OSC_10MHZ -> Net-(C18-Pad1)
- U1 pad 13: (no net) -> Net-(R9-Pad1)
- U1 pad 25: (no net) -> /BOARD_TEMP
- U1 pad 26: (no net) -> /LED_STATUS
- U1 pad 31: /OSC_10MHZ -> (no net)
- U1 pad 37: /LED_STATUS -> (no net)
- U1 pad 40: /OSC_10MHZ -> (no net)
- U1 pad 42: /GPS_1PPS -> (no net)
- U1 pad 63: /CPU_TO_AUX -> (no net)
- U1 pad 64: /AUX_TO_CPU -> (no net)
- U1 pad 67: (no net) -> /OSC_10MHZ
- U1 pad 69: (no net) -> /GPS_1PPS
- U1 pad 90: (no net) -> /OSC_10MHZ
- U5 pad 1: /USB_DP -> (no net)
- U5 pad 3: /USB_DM -> /USB_DP
- U5 pad 4: (no net) -> /USB_DM
Routing:
- net GND: track 0.00 -> 99.9 mm, vias 0 -> 185
- net Net-(AE5-Pad1): track 0.00 -> 96.1 mm
- net Net-(AE4-Pad1): track 0.00 -> 96.1 mm
- net Net-(AE3-Pad1): track 0.00 -> 96.1 mm
- net Net-(AE2-Pad1): track 0.00 -> 96.1 mm
- net +3V3: track 0.00 -> 56.6 mm, vias 0 -> 15
- net /SDA: track 0.00 -> 56.4 mm, vias 0 -> 2
- net /nRESET: track 0.00 -> 56.0 mm, vias 0 -> 1
- net /SCL: track 0.00 -> 55.2 mm, vias 0 -> 2
- net /OSC_10MHZ: track 0.00 -> 48.8 mm
- net /GPS_1PPS: track 0.00 -> 46.6 mm, vias 0 -> 3
- net /GPS_nRESET: track 0.00 -> 34.6 mm, vias 0 -> 2
- net /GPS_ONOFF: track 0.00 -> 30.4 mm, vias 0 -> 2
- net /BOARD_TEMP: track 0.00 -> 28.7 mm
- net /CPU_TO_GPS: track 0.00 -> 25.3 mm, vias 0 -> 2
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- added copper zone on In2.Cu, net +3V3
- added copper zone on B.Cu, net GND
- added copper zone on F.Cu, net GND
- added copper zone on In1.Cu, net GND
Other:
- copper layers 2 -> 4

Commit message: rotate
Parts:
- U5: footprint pace:srv05-4 -> pace:SOT-23-6L-srv05
Changed lines of the file:
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@@
     )
-  )
-  (module pace:srv05-4 (layer F.Cu)
-    (at 48.79 8.3)
-    (attr smd)
-    (fp_text reference U5 (at 0.18 -2.42) (layer F.SilkS)
-      (effects (font (size 1 1) (thickness 0.15)))
-    )
-    (fp_text value SRV05-4-newfp (at 0.11 2.44) (layer F.Fab)
-      (effects (font (size 1 1) (thickness 0.15)))
-    )
-    (fp_line (start -2 -1.5) (end -2 -1.36) (layer F.SilkS) (width 0.15))
-    (fp_line (start -1.5 -1.2) (end -1.2 -1.5) (layer F.Fab) (width 0.12))
-    (fp_line (start -1.2 -1.5) (end 1.5 -1.5) (layer F.Fab) (width 0.12))
-    (fp_line (start 1.5 -1.5) (end 1.5 1.5) (layer F.Fab) (width 0.12))
-    (fp_line (start -1.5 1.5) (end 1.5 1.5) (layer F.Fab) (width 0.12))
-    (fp_line (start -1.5 -1.2) (end -1.5 1.5) (layer F.Fab) (width 0.12))
-    (fp_line (start -1.5 -1.5) (end 1.5 -1.5) (layer F.SilkS) (width 0.15))
-    (fp_line (start -1.5 1.5) (end 1.5 1.5) (layer F.SilkS) (width 0.15))
-    (fp_line (start -1.5 -1.5) (end -2 -1.5) (layer F.SilkS) (width 0.15))
-    (fp_line (start -2 -1.53) (end -2 1.53) (layer F.CrtYd) (width 0.12))
-    (fp_line (start 2 1.53) (end -2 1.53) (layer F.CrtYd) (width 0.12))
-    (fp_line (start 2 -1.53) (end 2 1.53) (layer F.CrtYd) (width 0.12))
-    (fp_line (start -2 -1.53) (end 2 -1.53) (layer F.CrtYd) (width 0.12))
-    (pad 6 smd rect (at 1.2 -0.95) (size 1 0.7) (layers F.Cu F.Paste F.Mask))
-    (pad 5 smd rect (at 1.2 0) (size 1 0.7) (layers F.Cu F.Paste F.Mask)
-      (net 22 /VUSB))
-    (pad 4 smd rect (at 1.2 0.95) (size 1 0.7) (layers F.Cu F.Paste F.Mask)
-      (net 21 /USB_DM))
-    (pad 3 smd rect (at -1.2 0.95) (size 1 0.7) (layers F.Cu F.Paste F.Mask)
-      (net 23 /USB_DP))
-    (pad 2 smd rect (at -1.2 0) (size 1 0.7) (layers F.Cu F.Paste F.Mask)
-      (net 1 GND))
-    (pad 1 smd rect (at -1.2 -0.95) (size 1 0.7) (layers F.Cu F.Paste F.Mask))
   )
   (module LED_SMD:LED_0805_2012Metric (layer F.Cu)
@@
     )
   )
+  (module pace:SOT-23-6L-srv05 (layer F.Cu)
+    (at 48.79 8.3)
+    (attr smd)
+    (fp_text reference U5 (at 0.18 -2.42) (layer F.SilkS)
+      (effects (font (size 1 1) (thickness 0.15)))
+    )
+    (fp_text value SRV05-4-newfp (at 0.11 2.44) (layer F.Fab)
+      (effects (font (size 1 1) (thickness 0.15)))
+    )
+    (fp_line (start -2 -1.53) (end 2 -1.53) (layer F.CrtYd) (width 0.12))
+    (fp_line (start 2 -1.53) (end 2 1.53) (layer F.CrtYd) (width 0.12))
+    (fp_line (start 2 1.53) (end -2 1.53) (layer F.CrtYd) (width 0.12))
+    (fp_line (start -2 -1.53) (end -2 1.53) (layer F.CrtYd) (width 0.12))
+    (fp_line (start -1.5 -1.5) (end -2 -1.5) (layer F.SilkS) (width 0.15))
+    (fp_line (start -1.5 1.5) (end 1.5 1.5) (layer F.SilkS) (width 0.15))
+    (fp_line (start -1.5 -1.5) (end 1.5 -1.5) (layer F.SilkS) (width 0.15))
+    (fp_line (start -1.5 -1.2) (end -1.5 1.5) (layer F.Fab) (width 0.12))
+    (fp_line (start -1.5 1.5) (end 1.5 1.5) (layer F.Fab) (width 0.12))
+    (fp_line (start 1.5 -1.5) (end 1.5 1.5) (layer F.Fab) (width 0.12))
+    (fp_line (start -1.2 -1.5) (end 1.5 -1.5) (layer F.Fab) (width 0.12))
+    (fp_line (start -1.5 -1.2) (end -1.2 -1.5) (layer F.Fab) (width 0.12))
+    (fp_line (start -2 -1.5) (end -2 -1.36) (layer F.SilkS) (width 0.15))
+    (pad 1 smd rect (at -1.2 -0.95) (size 1 0.7) (layers F.Cu F.Paste F.Mask))
+    (pad 2 smd rect (at -1.2 0) (size 1 0.7) (layers F.Cu F.Paste F.Mask)
+      (net 1 GND))
+    (pad 3 smd rect (at -1.2 0.95) (size 1 0.7) (layers F.Cu F.Paste F.Mask)
+      (net 23 /USB_DP))
+    (pad 4 smd rect (at 1.2 0.95) (size 1 0.7) (layers F.Cu F.Paste F.Mask)
+      (net 21 /USB_DM))
+    (pad 5 smd rect (at 1.2 0) (size 1 0.7) (layers F.Cu F.Paste F.Mask)
+      (net 22 /VUSB))
+    (pad 6 smd rect (at 1.2 -0.95) (size 1 0.7) (layers F.Cu F.Paste F.Mask))
+  )
   (gr_line (start 0 0) (end 0 100) (layer Edge.Cuts) (width 0.05))
