File: gpsdo/gpsdo.kicad_pcb (KiCad board)
At the start: 4 copper layers, 100 x 100 mm, 64 parts, among them J1 Conn_02x05_Odd_Even, J2 Barrel_Jack_Switch, J3 usb-micro-jlc, J5 Conn_01x02_Male, SW1 pushbutton_switch, SW2 SW_SPDT, U1 STM32F407VETx, U2 ATGM336H-5N, U3 AP1117-33, U4 74AHC1G04-newfp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

Commit message: order
Parts:
- moved L1 3.45 mm to (81.4, 6.60)
- moved J3 2.56 mm to (48.5, 2.54)
- moved H3 0.41 mm to (3.50, 96.5)
- moved H2 0.32 mm to (3.50, 3.50)
- moved H1 0.14 mm to (96.5, 3.50)
- moved H4 0.10 mm to (96.5, 96.5)
Routing:
- net +3V3: track 56.6 -> 68.0 mm, vias 15 -> 20
- net GND: track 97.7 -> 90.5 mm, vias 185 -> 208
- net Net-(AE1-Pad1): track 13.3 -> 16.5 mm, vias 0 -> 2
- net Net-(C11-Pad1): track 8.16 -> 10.8 mm
- net Net-(L1-Pad1): track 6.22 -> 4.08 mm, vias 2 -> 0
Other:
- board text added: "*"
- board text added: "1PPS"
- board text added: "5-12v"
- board text added: "gpsdo 2021-03-01"
